Commit message: ursurg_description: Combine UR5e and LND tool (wip)

File: ursurg_description/urdf/eua.urdf.xacro (robot description, xacro)
@@ -2,6 +2,5 @@
 <robot name="eua" xmlns:xacro="http://ros.org/wiki/xacro">
   <xacro:macro name="eua1" params="prefix" >
-    <!-- <link name="${prefix}eua1_base" /> -->
-    <link name="${prefix}eua">
+    <link name="${prefix}eua1">
       <visual>
         <!-- <origin xyz="0 0 0" rpy="0 0 0" /> -->
@@ -15,3 +14,8 @@
     </link>
   </xacro:macro>
+  <xacro:macro name="eua2" params="prefix" >
+    <link name="${prefix}eua2">
+      <!-- TODO -->
+    </link>
+  </xacro:macro>
 </robot>

File: ursurg_description/urdf/ursurg.urdf.xacro (robot description, xacro)
@@ -1,6 +1,6 @@
 <?xml version="1.0"?>
 <robot name="a_ur5e_eua1_lnd420006" xmlns:xacro="http://ros.org/wiki/xacro">
-  <xacro:property name="prefix1" value="a_" />
-  <!-- <xacro:property name="prefix2" value="b_" /> -->
+  <xacro:include filename="eua.urdf.xacro" />
+  <xacro:include filename="lnd.urdf.xacro" />
   <link name="world" />
   <!-- UR5e robot
@@ -8,26 +8,63 @@
        kinematic configuration -->
   <xacro:include filename="$(find ur_e_description)/urdf/ur5e.urdf.xacro" />
-  <xacro:arg name="kinematics_config_file" default="$(find ur_e_description)/config/ur5e_default.yaml" />
-  <xacro:ur5e_robot prefix="${prefix1}ur_" joint_limited="false" kinematics_file="${load_yaml('$(arg kinematics_config_file)')}" />
-  <joint name="${prefix1}world_ur_base" type="fixed">
+  <xacro:arg name="ur5e_kinematics_config_file" default="$(find ur_e_description)/config/ur5e_default.yaml" />
+  <xacro:ur5e_robot prefix="a_ur_" joint_limited="false" kinematics_file="${load_yaml('$(arg ur5e_kinematics_config_file)')}" />
+  <joint name="a_world_ur_base_joint" type="fixed">
     <parent link="world" />
-    <child link="${prefix1}ur_base_link" />
-    <origin xyz="0 0 0" rpy="0 0 0" />
+    <child link="a_ur_base_link" />
+    <origin xyz="0.6 -0.2 0" rpy="0 0 ${-pi/2}" />
   </joint>
   <!-- EUA1 tool adapter -->
-  <xacro:include filename="eua.urdf.xacro" />
-  <xacro:eua1 prefix="${prefix1}" />
-  <joint name="${prefix1}ur_eua" type="fixed">
-    <parent link="${prefix1}ur_tool0" />
-    <child link="${prefix1}eua" />
+  <xacro:eua1 prefix="a_" />
+  <joint name="a_ur_eua_joint" type="fixed">
+    <parent link="a_ur_tool0" />
+    <child link="a_eua1" />
     <origin xyz="0 0 0.05" rpy="0 ${-pi/2} ${-pi/2}" />
   </joint>
   <!-- LND 420006 tool -->
-  <xacro:include filename="lnd.urdf.xacro" />
-  <xacro:lnd420006 prefix="${prefix1}tool_" />
-  <joint name="${prefix1}eua_tool" type="fixed">
-    <parent link="${prefix1}eua" />
-    <child link="${prefix1}tool_base" />
+  <xacro:lnd420006 prefix="a_tool_" />
+  <joint name="a_eua1_tool_joint" type="fixed">
+    <parent link="a_eua1" />
+    <child link="a_tool_base" />
     <origin xyz="0.015 0 0.055" rpy="0 0 0" />
   </joint>
+  <!-- UR5 robot -->
+  <xacro:include filename="$(find ur_description)/urdf/ur5.urdf.xacro" />
+  <xacro:arg name="ur5_kinematics_config_file" default="$(find ur_description)/config/ur5_default.yaml" />
+  <xacro:ur5_robot prefix="b_ur_" joint_limited="false" kinematics_file="${load_yaml('$(arg ur5_kinematics_config_file)')}" />
+  <joint name="b_world_ur_base_joint" type="fixed">
+    <parent link="world" />
+    <child link="b_ur_base_link" />
+    <origin xyz="0.6 -1 0" rpy="0 0 ${-pi/2}" />
+  </joint>
+  <!-- EUA2 tool adapter -->
+  <xacro:eua2 prefix="b_" />
+  <joint name="b_ur_eua2_joint" type="fixed">
+    <parent link="b_ur_tool0" />
+    <child link="b_eua2" />
+    <origin xyz="0 0 0.05" rpy="0 ${-pi/2} ${-pi/2}" />
+  </joint>
+  <!-- LND 470006 tool -->
+  <xacro:lnd470006 prefix="b_tool_" />
+  <joint name="b_eua2_tool_joint" type="fixed">
+    <parent link="b_eua2" />
+    <child link="b_tool_base" />
+    <origin xyz="0.015 0 0.055" rpy="0 0 0" />
+  </joint>
+  <!-- Table -->
+  <link name="table_base">
+    <visual>
+      <origin xyz="0.4 -0.6 -0.4" rpy="0 0 ${pi/2}" />
+      <geometry>
+        <box size="1.2 0.8 0.8" />
+      </geometry>
+      <material name="table_color">
+        <color rgba="0.55 0.45 0.3 1.0" />
+      </material>
+    </visual>
+  </link>
+  <joint name="world_table_base_joint" type="fixed">
+    <parent link="world" />
+    <child link="table_base" />
+  </joint>
 </robot>

Commit message: ursurg_description: Complete model
Still todo: EUA2 dimensions

File: ursurg_description/urdf/eua.urdf.xacro (robot description, xacro)
@@ -2,7 +2,7 @@
 <robot name="eua" xmlns:xacro="http://ros.org/wiki/xacro">
   <xacro:macro name="eua1" params="prefix" >
-    <link name="${prefix}eua1">
+    <link name="${prefix}eua1_robot_mount" />
+    <link name="${prefix}eua1_base">
       <visual>
-        <!-- <origin xyz="0 0 0" rpy="0 0 0" /> -->
         <geometry>
           <box size="0.07 0.17 0.08" />
@@ -13,9 +13,31 @@
       </visual>
     </link>
+    <link name="${prefix}eua1_tool_mount" />
+    <joint name="${prefix}eua1_robot_mount_base_joint" type="fixed">
+      <parent link="${prefix}eua1_robot_mount" />
+      <child link="${prefix}eua1_base" />
+      <origin xyz="0.035 0 0.04" rpy="0 ${-pi/2} ${-pi/2}" />
+    </joint>
+    <joint name="${prefix}eua1_base_tool_mount_joint" type="fixed">
+      <parent link="${prefix}eua1_base" />
+      <child link="${prefix}eua1_tool_mount" />
+      <origin xyz="0 0 0.04" rpy="0 0 0" />
+    </joint>
   </xacro:macro>
   <xacro:macro name="eua2" params="prefix" >
-    <link name="${prefix}eua2">
+    <link name="${prefix}eua2_robot_mount" />
+    <link name="${prefix}eua2_base">
       <!-- TODO -->
     </link>
+    <link name="${prefix}eua2_tool_mount" />
+    <joint name="${prefix}eua2_robot_mount_base_joint" type="fixed">
+      <parent link="${prefix}eua2_robot_mount" />
+      <child link="${prefix}eua2_base" />
+      <origin xyz="0 0 0.08" rpy="0 ${-pi/2} ${pi/2}" />
+    </joint>
+    <joint name="${prefix}eua2_base_tool_mount_joint" type="fixed">
+      <parent link="${prefix}eua2_base" />
+      <child link="${prefix}eua2_tool_mount" />
+    </joint>
   </xacro:macro>
 </robot>

File: ursurg_description/urdf/lnd.urdf.xacro (robot description, xacro)
@@ -93,4 +93,5 @@
   </xacro:macro>
   <xacro:macro name="lnd420006" params="prefix">
+    <link name="${prefix}mount" />
     <link name="${prefix}base">
       <visual>
@@ -111,7 +112,13 @@
       </visual>
     </link>
+    <joint name="${prefix}base_mount_joint" type="fixed">
+      <parent link="${prefix}mount" />
+      <child link="${prefix}base" />
+      <origin xyz="0.015 0 0.015" rpy="0 0 0" />
+    </joint>
     <xacro:lnd_tip prefix="${prefix}" d="0.467" />
   </xacro:macro>
   <xacro:macro name="lnd470006" params="prefix">
+    <link name="${prefix}mount" />
     <link name="${prefix}base">
       <visual>
@@ -132,4 +139,9 @@
       </visual>
     </link>
+    <joint name="${prefix}base_mount_joint" type="fixed">
+      <parent link="${prefix}mount" />
+      <child link="${prefix}base" />
+      <origin xyz="-0.015 0 0.021" rpy="0 0 0" />
+    </joint>
     <xacro:lnd_tip prefix="${prefix}" d="0.5435" />
   </xacro:macro>

File: ursurg_description/urdf/ursurg.urdf.xacro (robot description, xacro)
@@ -4,5 +4,5 @@
   <xacro:include filename="lnd.urdf.xacro" />
   <link name="world" />
-  <!-- UR5e robot
+  <!-- A) UR5e robot
        Run xacro with arg 'kinematics_config_file' set to override the default
        kinematic configuration -->
@@ -13,21 +13,19 @@
     <parent link="world" />
     <child link="a_ur_base_link" />
-    <origin xyz="0.6 -0.2 0" rpy="0 0 ${-pi/2}" />
+    <origin xyz="0.6 -0.2 0" rpy="0 0 ${pi/2}" />
   </joint>
-  <!-- EUA1 tool adapter -->
+  <!-- A) EUA1 tool adapter -->
   <xacro:eua1 prefix="a_" />
   <joint name="a_ur_eua_joint" type="fixed">
     <parent link="a_ur_tool0" />
-    <child link="a_eua1" />
-    <origin xyz="0 0 0.05" rpy="0 ${-pi/2} ${-pi/2}" />
+    <child link="a_eua1_robot_mount" />
   </joint>
-  <!-- LND 420006 tool -->
+  <!-- A) LND 420006 tool -->
   <xacro:lnd420006 prefix="a_tool_" />
   <joint name="a_eua1_tool_joint" type="fixed">
-    <parent link="a_eua1" />
-    <child link="a_tool_base" />
-    <origin xyz="0.015 0 0.055" rpy="0 0 0" />
+    <parent link="a_eua1_tool_mount" />
+    <child link="a_tool_mount" />
   </joint>
-  <!-- UR5 robot -->
+  <!-- B) UR5 robot -->
   <xacro:include filename="$(find ur_description)/urdf/ur5.urdf.xacro" />
   <xacro:arg name="ur5_kinematics_config_file" default="$(find ur_description)/config/ur5_default.yaml" />
@@ -36,19 +34,18 @@
     <parent link="world" />
     <child link="b_ur_base_link" />
-    <origin xyz="0.6 -1 0" rpy="0 0 ${-pi/2}" />
+    <origin xyz="0.6 -1 0" rpy="0 0 ${pi/2}" />
   </joint>
-  <!-- EUA2 tool adapter -->
+  <!-- B) EUA2 tool adapter -->
   <xacro:eua2 prefix="b_" />
   <joint name="b_ur_eua2_joint" type="fixed">
     <parent link="b_ur_tool0" />
-    <child link="b_eua2" />
-    <origin xyz="0 0 0.05" rpy="0 ${-pi/2} ${-pi/2}" />
+    <child link="b_eua2_robot_mount" />
   </joint>
-  <!-- LND 470006 tool -->
+  <!-- B) LND 470006 tool -->
   <xacro:lnd470006 prefix="b_tool_" />
   <joint name="b_eua2_tool_joint" type="fixed">
-    <parent link="b_eua2" />
-    <child link="b_tool_base" />
-    <origin xyz="0.015 0 0.055" rpy="0 0 0" />
+    <parent link="b_eua2_tool_mount" />
+    <child link="b_tool_mount" />
+    <!-- <origin xyz="0.015 0 0.055" rpy="0 0 0" /> -->
   </joint>
   <!-- Table -->

Commit message: description: Remove hard-coded euaX_ prefix

File: ursurg_description/urdf/eua.urdf.xacro (robot description, xacro)
@@ -2,6 +2,6 @@
 <robot name="eua" xmlns:xacro="http://ros.org/wiki/xacro">
   <xacro:macro name="eua1" params="prefix" >
-    <link name="${prefix}eua1_robot_mount" />
-    <link name="${prefix}eua1_base">
+    <link name="${prefix}robot_mount" />
+    <link name="${prefix}base">
       <visual>
         <geometry>
@@ -13,30 +13,30 @@
       </visual>
     </link>
-    <link name="${prefix}eua1_tool_mount" />
-    <joint name="${prefix}eua1_robot_mount_base_joint" type="fixed">
-      <parent link="${prefix}eua1_robot_mount" />
-      <child link="${prefix}eua1_base" />
+    <link name="${prefix}tool_mount" />
+    <joint name="${prefix}robot_mount_base_joint" type="fixed">
+      <parent link="${prefix}robot_mount" />
+      <child link="${prefix}base" />
       <origin xyz="0.035 0 0.04" rpy="0 ${-pi/2} ${-pi/2}" />
     </joint>
-    <joint name="${prefix}eua1_base_tool_mount_joint" type="fixed">
-      <parent link="${prefix}eua1_base" />
-      <child link="${prefix}eua1_tool_mount" />
+    <joint name="${prefix}base_tool_mount_joint" type="fixed">
+      <parent link="${prefix}base" />
+      <child link="${prefix}tool_mount" />
       <origin xyz="0 0 0.04" rpy="0 0 0" />
     </joint>
   </xacro:macro>
   <xacro:macro name="eua2" params="prefix" >
-    <link name="${prefix}eua2_robot_mount" />
-    <link name="${prefix}eua2_base">
+    <link name="${prefix}robot_mount" />
+    <link name="${prefix}base">
       <!-- TODO -->
     </link>
-    <link name="${prefix}eua2_tool_mount" />
-    <joint name="${prefix}eua2_robot_mount_base_joint" type="fixed">
-      <parent link="${prefix}eua2_robot_mount" />
-      <child link="${prefix}eua2_base" />
+    <link name="${prefix}tool_mount" />
+    <joint name="${prefix}robot_mount_base_joint" type="fixed">
+      <parent link="${prefix}robot_mount" />
+      <child link="${prefix}base" />
       <origin xyz="0 0 0.08" rpy="0 ${-pi/2} ${pi/2}" />
     </joint>
-    <joint name="${prefix}eua2_base_tool_mount_joint" type="fixed">
-      <parent link="${prefix}eua2_base" />
-      <child link="${prefix}eua2_tool_mount" />
+    <joint name="${prefix}base_tool_mount_joint" type="fixed">
+      <parent link="${prefix}base" />
+      <child link="${prefix}tool_mount" />
     </joint>
   </xacro:macro>
