Commit message: ursurg_description: Combine UR5e and LND tool (wip)

File: ursurg_description/urdf/lnd.urdf.xacro (robot description, xacro)
@@ -5,5 +5,8 @@
     <color rgba="0.667 0.663 0.678 1.0" />
   </material>
-  <xacro:macro name="lnd_tip" params="prefix">
+  <material name="rod_dark_grey">
+    <color rgba="0.1 0.1 0.1 1.0" />
+  </material>
+  <xacro:macro name="lnd_tip" params="prefix d" >
     <link name="${prefix}roll">
       <visual>
@@ -48,5 +51,5 @@
       <parent link="${prefix}base" />
       <child link="${prefix}roll" />
-      <origin xyz="0.467 0 0" rpy="${-pi} ${-pi/2} 0" />
+      <origin xyz="${d} 0 0" rpy="${-pi} ${-pi/2} 0" />
       <axis xyz="0 0 1" />
       <limit lower="${radians(-260)}" upper="${radians(260)}" effort="5" velocity="${pi}" />
@@ -69,5 +72,5 @@
       <origin xyz="0 0 0" rpy="0 0 0" />
       <axis xyz="0 0 1" />
-      <limit lower="${radians(-10)}" upper="${radians(75)}" effort="5" velocity="${pi}" />
+      <limit lower="0" upper="${radians(75)}" effort="5" velocity="${pi}" />
     </joint>
     <joint name="${prefix}jaw2_joint" type="revolute">
@@ -76,5 +79,5 @@
       <origin xyz="0 0 0" rpy="${pi} 0 0" />
       <axis xyz="0 0 1" />
-      <limit lower="${radians(-10)}" upper="${radians(75)}" effort="5" velocity="${pi}" />
+      <limit lower="0" upper="${radians(75)}" effort="5" velocity="${pi}" />
     </joint>
     <joint name="${prefix}tcp1_joint" type="fixed">
@@ -105,15 +108,29 @@
           <cylinder radius="0.004" length="0.457" />
         </geometry>
-        <material name="rod_dark_grey">
-          <color rgba="0.1 0.1 0.1 1.0" />
+        <material name="rod_dark_grey" />
+      </visual>
+    </link>
+    <xacro:lnd_tip prefix="${prefix}" d="0.467" />
+  </xacro:macro>
+  <xacro:macro name="lnd470006" params="prefix">
+    <link name="${prefix}base">
+      <visual>
+        <origin xyz="-0.015 0 -0.019" rpy="0 0 0" />
+        <geometry>
+          <box size="0.06 0.045 0.08" />
+        </geometry>
+        <material name="housing_white">
+          <color rgba="1.0 1.0 1.0 1.0" />
         </material>
       </visual>
+      <visual>
+        <origin xyz="0.26675 0 0" rpy="0 ${pi/2} 0" />
+        <geometry>
+          <cylinder radius="0.004" length="0.5335" />
+        </geometry>
+        <material name="rod_dark_grey" />
+      </visual>
     </link>
-    <xacro:lnd_tip prefix="${prefix}" />
-  </xacro:macro>
-  <xacro:macro name="lnd470006" params="prefix">
-    <!-- TODO -->
-    <link name="${prefix}base"></link>
-    <xacro:lnd_tip prefix="${prefix}" />
+    <xacro:lnd_tip prefix="${prefix}" d="0.5435" />
   </xacro:macro>
 </robot>

Commit message: Fix LND joint names

File: ursurg_description/urdf/lnd.urdf.xacro (robot description, xacro)
@@ -9,5 +9,5 @@
   </material>
   <xacro:macro name="lnd_tip" params="prefix d" >
-    <link name="${prefix}roll">
+    <link name="${prefix}lower_rod">
       <visual>
         <origin xyz="0 0 -0.01" rpy="0 0 ${pi/2}" />
@@ -48,13 +48,13 @@
     <link name="${prefix}tcp1" />
     <link name="${prefix}tcp2" />
-    <joint name="${prefix}roll_joint" type="revolute">
+    <joint name="${prefix}roll" type="revolute">
       <parent link="${prefix}base" />
-      <child link="${prefix}roll" />
+      <child link="${prefix}lower_rod" />
       <origin xyz="${d} 0 0" rpy="${-pi} ${-pi/2} 0" />
       <axis xyz="0 0 1" />
       <limit lower="${radians(-260)}" upper="${radians(260)}" effort="5" velocity="${pi}" />
     </joint>
-    <joint name="${prefix}wrist_joint" type="revolute">
-      <parent link="${prefix}roll" />
+    <joint name="${prefix}pitch" type="revolute">
+      <parent link="${prefix}lower_rod" />
       <child link="${prefix}wrist" />
       <origin xyz="0 0 0" rpy="${-pi/2} ${-pi/2} 0" />
@@ -62,10 +62,10 @@
       <limit lower="${radians(-75)}" upper="${radians(75)}" effort="5" velocity="${pi}" />
     </joint>
-    <joint name="${prefix}jaw0_joint" type="fixed">
+    <joint name="${prefix}jaw0_fixed" type="fixed">
       <parent link="${prefix}wrist" />
       <child link="${prefix}jaw0" />
       <origin xyz="0.0091 0 0" rpy="${pi/2} 0 0" />
     </joint>
-    <joint name="${prefix}jaw1_joint" type="revolute">
+    <joint name="${prefix}yaw1" type="revolute">
       <parent link="${prefix}jaw0" />
       <child link="${prefix}jaw1" />
@@ -74,5 +74,5 @@
       <limit lower="0" upper="${radians(75)}" effort="5" velocity="${pi}" />
     </joint>
-    <joint name="${prefix}jaw2_joint" type="revolute">
+    <joint name="${prefix}yaw2" type="revolute">
       <parent link="${prefix}jaw0" />
       <child link="${prefix}jaw2" />
@@ -81,10 +81,10 @@
       <limit lower="0" upper="${radians(75)}" effort="5" velocity="${pi}" />
     </joint>
-    <joint name="${prefix}tcp1_joint" type="fixed">
+    <joint name="${prefix}tcp1_fixed" type="fixed">
       <parent link="${prefix}jaw1" />
       <child link="${prefix}tcp1" />
       <origin xyz="0.009 0 0" rpy="0 0 0" />
     </joint>
-    <joint name="${prefix}tcp2_joint" type="fixed">
+    <joint name="${prefix}tcp2_fixed" type="fixed">
       <parent link="${prefix}jaw2" />
       <child link="${prefix}tcp2" />

Commit message: description: Refactor to allow for robot-ee to tool-tip calibration

File: ursurg_description/urdf/lnd.urdf.xacro (robot description, xacro)
@@ -8,6 +8,7 @@
     <color rgba="0.1 0.1 0.1 1.0" />
   </material>
-  <xacro:macro name="lnd_tip" params="prefix d" >
-    <link name="${prefix}lower_rod">
+  <xacro:macro name="lnd_tip" params="prefix" >
+    <link name="${prefix}tip_calib" />
+    <link name="${prefix}rotation">
       <visual>
         <origin xyz="0 0 -0.01" rpy="0 0 ${pi/2}" />
@@ -49,12 +50,12 @@
     <link name="${prefix}tcp2" />
     <joint name="${prefix}roll" type="revolute">
-      <parent link="${prefix}base" />
-      <child link="${prefix}lower_rod" />
-      <origin xyz="${d} 0 0" rpy="${-pi} ${-pi/2} 0" />
+      <parent link="${prefix}tip_calib" />
+      <child link="${prefix}rotation" />
+      <origin xyz="-0.018 0 0" rpy="${-pi} ${-pi/2} 0" />
       <axis xyz="0 0 1" />
       <limit lower="${radians(-260)}" upper="${radians(260)}" effort="5" velocity="${pi}" />
     </joint>
     <joint name="${prefix}pitch" type="revolute">
-      <parent link="${prefix}lower_rod" />
+      <parent link="${prefix}rotation" />
       <child link="${prefix}wrist" />
       <origin xyz="0 0 0" rpy="${-pi/2} ${-pi/2} 0" />
@@ -93,8 +94,21 @@
   </xacro:macro>
   <xacro:macro name="lnd420006" params="prefix">
-    <link name="${prefix}mount" />
-    <link name="${prefix}base">
+    <xacro:lnd_tip prefix="${prefix}" />
+    <link name="${prefix}rod">
       <visual>
-        <origin xyz="-0.015 0 0" rpy="0 0 0" />
+        <geometry>
+          <cylinder radius="0.004" length="0.457" />
+        </geometry>
+        <material name="rod_dark_grey" />
+      </visual>
+    </link>
+    <joint name="${prefix}rod_joint" type="fixed">
+      <parent link="${prefix}rotation" />
+      <child link="${prefix}rod" />
+      <origin xyz="0 0 ${-0.457/2 - 0.01}" rpy="0 0 0" />
+    </joint>
+    <link name="${prefix}housing">
+      <visual>
+        <origin xyz="-0.013 0 0" rpy="0 0 0" />
         <geometry>
           <box size="0.096 0.065 0.03" />
@@ -104,22 +118,27 @@
         </material>
       </visual>
+    </link>
+    <joint name="${prefix}housing_joint" type="fixed">
+      <parent link="${prefix}tip_calib" />
+      <child link="${prefix}housing" />
+      <origin xyz="${-0.018 - 0.01 - 0.457} 0 0" rpy="0 0 0" />
+    </joint>
+  </xacro:macro>
+  <xacro:macro name="lnd470006" params="prefix">
+    <xacro:lnd_tip prefix="${prefix}" />
+    <link name="${prefix}rod">
       <visual>
-        <origin xyz="0.2285 0 0" rpy="0 ${pi/2} 0" />
         <geometry>
-          <cylinder radius="0.004" length="0.457" />
+          <cylinder radius="0.004" length="0.5335" />
         </geometry>
         <material name="rod_dark_grey" />
       </visual>
     </link>
-    <joint name="${prefix}base_mount_joint" type="fixed">
-      <parent link="${prefix}mount" />
-      <child link="${prefix}base" />
-      <origin xyz="0.015 0 0.015" rpy="0 0 0" />
+    <joint name="${prefix}rod_joint" type="fixed">
+      <parent link="${prefix}rotation" />
+      <child link="${prefix}rod" />
+      <origin xyz="0 0 ${-0.5335/2 - 0.01}" rpy="0 0 0" />
     </joint>
-    <xacro:lnd_tip prefix="${prefix}" d="0.467" />
-  </xacro:macro>
-  <xacro:macro name="lnd470006" params="prefix">
-    <link name="${prefix}mount" />
-    <link name="${prefix}base">
+    <link name="${prefix}housing">
       <visual>
         <origin xyz="-0.015 0 -0.019" rpy="0 0 0" />
@@ -131,18 +150,10 @@
         </material>
       </visual>
-      <visual>
-        <origin xyz="0.26675 0 0" rpy="0 ${pi/2} 0" />
-        <geometry>
-          <cylinder radius="0.004" length="0.5335" />
-        </geometry>
-        <material name="rod_dark_grey" />
-      </visual>
     </link>
-    <joint name="${prefix}base_mount_joint" type="fixed">
-      <parent link="${prefix}mount" />
-      <child link="${prefix}base" />
-      <origin xyz="-0.015 0 0.021" rpy="0 0 0" />
+    <joint name="${prefix}housing_joint" type="fixed">
+      <parent link="${prefix}tip_calib" />
+      <child link="${prefix}housing" />
+      <origin xyz="${-0.018 - 0.01 - 0.5335} 0 0" rpy="0 0 0" />
     </joint>
-    <xacro:lnd_tip prefix="${prefix}" d="0.5435" />
   </xacro:macro>
 </robot>

File: ursurg_description/urdf/ursurg.urdf.xacro (robot description, xacro)
@@ -18,7 +18,7 @@
   <joint name="a_ur_tool_joint" type="fixed">
     <parent link="a_ur_ee_link" />
-    <child link="a_tool_mount" />
+    <child link="a_tool_tip_calib" />
     <!-- TODO: Calibrate to find this transform accurately -->
-    <origin xyz="0.09 0 0" rpy="${pi} 0 0" />
+    <origin xyz="0.66 0 0" rpy="0 0 0" />
   </joint>
   <!-- B) UR5 robot -->
@@ -35,7 +35,6 @@
   <joint name="b_eua2_tool_joint" type="fixed">
     <parent link="b_ur_ee_link" />
-    <child link="b_tool_mount" />
-    <!-- TODO: Calibrate to find this transform accurately -->
-    <origin xyz="0.075 0 0.04" rpy="0 0 0" />
+    <child link="b_tool_tip_calib" />
+    <origin xyz="0.56961 -0.0012618 0.056071" rpy="0 0 0" /> <!-- From calibration -->
   </joint>
   <!-- Touch haptic devices -->

Commit message: description: Adjust LND joint limits

File: ursurg_description/urdf/lnd.urdf.xacro (robot description, xacro)
@@ -54,5 +54,5 @@
       <origin xyz="-0.018 0 0" rpy="${-pi} ${-pi/2} 0" />
       <axis xyz="0 0 1" />
-      <limit lower="${radians(-260)}" upper="${radians(260)}" effort="5" velocity="${pi}" />
+      <limit lower="${radians(-260)}" upper="${radians(260)}" effort="0.3" velocity="${2*pi}" />
     </joint>
     <joint name="${prefix}pitch" type="revolute">
@@ -61,5 +61,5 @@
       <origin xyz="0 0 0" rpy="${-pi/2} ${-pi/2} 0" />
       <axis xyz="0 0 1" />
-      <limit lower="${radians(-75)}" upper="${radians(75)}" effort="5" velocity="${pi}" />
+      <limit lower="${radians(-80)}" upper="${radians(80)}" effort="0.25" velocity="${2*pi}" />
     </joint>
     <joint name="${prefix}jaw0_fixed" type="fixed">
@@ -73,5 +73,5 @@
       <origin xyz="0 0 0" rpy="0 0 0" />
       <axis xyz="0 0 1" />
-      <limit lower="0" upper="${radians(75)}" effort="5" velocity="${pi}" />
+      <limit lower="${radians(-40)}" upper="${radians(80)}" effort="0.2" velocity="${2*pi}" />
     </joint>
     <joint name="${prefix}yaw2" type="revolute">
@@ -80,5 +80,5 @@
       <origin xyz="0 0 0" rpy="${pi} 0 0" />
       <axis xyz="0 0 1" />
-      <limit lower="0" upper="${radians(75)}" effort="5" velocity="${pi}" />
+      <limit lower="${radians(-40)}" upper="${radians(80)}" effort="0.2" velocity="${2*pi}" />
     </joint>
     <joint name="${prefix}tcp1_fixed" type="fixed">

Commit message: Increase jaw/TCP joint limits

File: ursurg_description/urdf/lnd.urdf.xacro (robot description, xacro)
@@ -73,5 +73,5 @@
       <origin xyz="0 0 0" rpy="0 0 0" />
       <axis xyz="0 0 1" />
-      <limit lower="${radians(-40)}" upper="${radians(80)}" effort="0.2" velocity="${2*pi}" />
+      <limit lower="${radians(-75)}" upper="${radians(75)}" effort="0.2" velocity="${2*pi}" />
     </joint>
     <joint name="${prefix}yaw2" type="revolute">
@@ -80,5 +80,5 @@
       <origin xyz="0 0 0" rpy="${pi} 0 0" />
       <axis xyz="0 0 1" />
-      <limit lower="${radians(-40)}" upper="${radians(80)}" effort="0.2" velocity="${2*pi}" />
+      <limit lower="${radians(-75)}" upper="${radians(75)}" effort="0.2" velocity="${2*pi}" />
     </joint>
     <joint name="${prefix}tcp1_fixed" type="fixed">

Commit message: state_publisher: Publish TCP pose and grasper angle and put TCP frame in URDF

File: ursurg_description/urdf/lnd.urdf.xacro (robot description, xacro)
@@ -28,4 +28,5 @@
       </visual>
     </link>
+    <link name="${prefix}jaw_hinge" />
     <link name="${prefix}jaw0" />
     <link name="${prefix}jaw1">
@@ -47,4 +48,5 @@
       </visual>
     </link>
+    <link name="${prefix}tcp0" />
     <link name="${prefix}tcp1" />
     <link name="${prefix}tcp2" />
@@ -63,11 +65,19 @@
       <limit lower="${radians(-80)}" upper="${radians(80)}" effort="0.25" velocity="${2*pi}" />
     </joint>
-    <joint name="${prefix}jaw0_fixed" type="fixed">
+    <joint name="${prefix}jaw_hinge_fixed" type="fixed">
       <parent link="${prefix}wrist" />
-      <child link="${prefix}jaw0" />
+      <child link="${prefix}jaw_hinge" />
       <origin xyz="0.0091 0 0" rpy="${pi/2} 0 0" />
     </joint>
+    <!-- This is not a real physical joint, but rather yaw0 = (yaw1 - yaw2) / 2,
+         ie. the TCP frame is at an angle between the grasper jaws. -->
+    <joint name="${prefix}yaw0" type="continuous">
+      <parent link="${prefix}jaw_hinge" />
+      <child link="${prefix}jaw0" />
+      <origin xyz="0 0 0" rpy="0 0 0" />
+      <axis xyz="0 0 1" />
+    </joint>
     <joint name="${prefix}yaw1" type="revolute">
-      <parent link="${prefix}jaw0" />
+      <parent link="${prefix}jaw_hinge" />
       <child link="${prefix}jaw1" />
       <origin xyz="0 0 0" rpy="0 0 0" />
@@ -76,9 +86,14 @@
     </joint>
     <joint name="${prefix}yaw2" type="revolute">
-      <parent link="${prefix}jaw0" />
+      <parent link="${prefix}jaw_hinge" />
       <child link="${prefix}jaw2" />
       <origin xyz="0 0 0" rpy="${pi} 0 0" />
       <axis xyz="0 0 1" />
       <limit lower="${radians(-75)}" upper="${radians(75)}" effort="0.2" velocity="${2*pi}" />
+    </joint>
+    <joint name="${prefix}tcp0_fixed" type="fixed">
+      <parent link="${prefix}jaw0" />
+      <child link="${prefix}tcp0" />
+      <origin xyz="0.009 0 0" rpy="0 0 0" />
     </joint>
     <joint name="${prefix}tcp1_fixed" type="fixed">

Commit message: ursurg_description: Change LND yaw0 to revolute type to include limits

File: ursurg_description/urdf/lnd.urdf.xacro (robot description, xacro)
@@ -72,9 +72,10 @@
     <!-- This is not a real physical joint, but rather yaw0 = (yaw1 - yaw2) / 2,
          ie. the TCP frame is at an angle between the grasper jaws. -->
-    <joint name="${prefix}yaw0" type="continuous">
+    <joint name="${prefix}yaw0" type="revolute">
       <parent link="${prefix}jaw_hinge" />
       <child link="${prefix}jaw0" />
       <origin xyz="0 0 0" rpy="0 0 0" />
       <axis xyz="0 0 1" />
+      <limit lower="${radians(-75)}" upper="${radians(75)}" effort="0.2" velocity="${2*pi}" />
     </joint>
     <joint name="${prefix}yaw1" type="revolute">
