Commit message: description: Don't include EUAs for now
And never in kinematic chain. Including EUA geometry in the
future will be nice for collision checking however.

File: ursurg_description/urdf/ursurg.urdf.xacro (robot description, xacro)
@@ -15,15 +15,11 @@
     <origin xyz="0.6 -0.2 0" rpy="0 0 ${pi/2}" />
   </joint>
-  <!-- A) EUA1 tool adapter -->
-  <xacro:eua1 prefix="a_" />
-  <joint name="a_ur_eua_joint" type="fixed">
-    <parent link="a_ur_tool0" />
-    <child link="a_eua1_robot_mount" />
-  </joint>
   <!-- A) LND 420006 tool -->
   <xacro:lnd420006 prefix="a_tool_" />
-  <joint name="a_eua1_tool_joint" type="fixed">
-    <parent link="a_eua1_tool_mount" />
+  <joint name="a_ur_tool_joint" type="fixed">
+    <parent link="a_ur_tool0" />
     <child link="a_tool_mount" />
+    <!-- TODO: Measure/calibrate to find this transform accurately -->
+    <origin xyz="0 0.035 0.08" rpy="0 ${-pi/2} ${-pi/2}" />
   </joint>
   <!-- B) UR5 robot -->
@@ -36,16 +32,11 @@
     <origin xyz="0.6 -1 0" rpy="0 0 ${pi/2}" />
   </joint>
-  <!-- B) EUA2 tool adapter -->
-  <xacro:eua2 prefix="b_" />
-  <joint name="b_ur_eua2_joint" type="fixed">
-    <parent link="b_ur_tool0" />
-    <child link="b_eua2_robot_mount" />
-  </joint>
   <!-- B) LND 470006 tool -->
   <xacro:lnd470006 prefix="b_tool_" />
   <joint name="b_eua2_tool_joint" type="fixed">
-    <parent link="b_eua2_tool_mount" />
+    <parent link="b_ur_tool0" />
     <child link="b_tool_mount" />
-    <!-- <origin xyz="0.015 0 0.055" rpy="0 0 0" /> -->
+    <!-- TODO: Measure/calibrate to find this transform accurately -->
+    <origin xyz="0 0 0.12" rpy="0 ${-pi/2} ${-pi/2}" />
   </joint>
   <!-- Table -->

Commit message: description: Use the ee_link of the UR's for attaching tools

File: ursurg_description/urdf/ursurg.urdf.xacro (robot description, xacro)
@@ -18,8 +18,8 @@
   <xacro:lnd420006 prefix="a_tool_" />
   <joint name="a_ur_tool_joint" type="fixed">
-    <parent link="a_ur_tool0" />
+    <parent link="a_ur_ee_link" />
     <child link="a_tool_mount" />
     <!-- TODO: Measure/calibrate to find this transform accurately -->
-    <origin xyz="0 0.035 0.08" rpy="0 ${-pi/2} ${-pi/2}" />
+    <origin xyz="0.08 0 -0.035" rpy="${pi} 0 0" />
   </joint>
   <!-- B) UR5 robot -->
@@ -35,8 +35,8 @@
   <xacro:lnd470006 prefix="b_tool_" />
   <joint name="b_eua2_tool_joint" type="fixed">
-    <parent link="b_ur_tool0" />
+    <parent link="b_ur_ee_link" />
     <child link="b_tool_mount" />
     <!-- TODO: Measure/calibrate to find this transform accurately -->
-    <origin xyz="0 0 0.12" rpy="0 ${-pi/2} ${-pi/2}" />
+    <origin xyz="0.1 0 0" rpy="${pi} 0 0" />
   </joint>
   <!-- Table -->

Commit message: description: Update tool-robot transform with measured values

File: ursurg_description/urdf/ursurg.urdf.xacro (robot description, xacro)
@@ -1,5 +1,4 @@
 <?xml version="1.0"?>
-<robot name="a_ur5e_eua1_lnd420006" xmlns:xacro="http://ros.org/wiki/xacro">
-  <xacro:include filename="eua.urdf.xacro" />
+<robot name="ursurg" xmlns:xacro="http://ros.org/wiki/xacro">
   <xacro:include filename="lnd.urdf.xacro" />
   <link name="world" />
@@ -20,6 +19,6 @@
     <parent link="a_ur_ee_link" />
     <child link="a_tool_mount" />
-    <!-- TODO: Measure/calibrate to find this transform accurately -->
-    <origin xyz="0.08 0 -0.035" rpy="${pi} 0 0" />
+    <!-- TODO: Calibrate to find this transform accurately -->
+    <origin xyz="0.075 0 -0.04" rpy="${pi} 0 0" />
   </joint>
   <!-- B) UR5 robot -->
@@ -37,6 +36,6 @@
     <parent link="b_ur_ee_link" />
     <child link="b_tool_mount" />
-    <!-- TODO: Measure/calibrate to find this transform accurately -->
-    <origin xyz="0.1 0 0" rpy="${pi} 0 0" />
+    <!-- TODO: Calibrate to find this transform accurately -->
+    <origin xyz="0.09 0 0" rpy="${pi} 0 0" />
   </joint>
   <!-- Table -->

Commit message: description: Add Touch haptic devices to ursurg scene

File: ursurg_description/urdf/ursurg.urdf.xacro (robot description, xacro)
@@ -55,3 +55,24 @@
     <child link="table_base" />
   </joint>
+  <!-- Touch haptic devices -->
+  <xacro:property name="touch_descr" value="$(find touch_description)/urdf/touch.urdf.xacro" />
+  <xacro:if value="${len(touch_descr) == 0}">
+    <link name="touch_left_base" />
+    <link name="touch_right_base" />
+  </xacro:if>
+  <xacro:unless value="${len(touch_descr) == 0}">
+    <xacro:include filename="${touch_descr}" />
+    <xacro:touch prefix="touch_left_" />
+    <xacro:touch prefix="touch_right_" />
+  </xacro:unless>
+  <joint name="world_touch_left_fixed" type="fixed">
+    <parent link="world" />
+    <child link="touch_left_base" />
+    <origin xyz="-0.6 -0.5 0" rpy="0 0 ${pi/2}" />
+  </joint>
+  <joint name="world_touch_right_fixed" type="fixed">
+    <parent link="world" />
+    <child link="touch_right_base" />
+    <origin xyz="-0.6 -0.7 0" rpy="0 0 ${pi/2}" />
+  </joint>
 </robot>

Commit message: description: Include only touch base frames and not the 3D model

File: ursurg_description/urdf/ursurg.urdf.xacro (robot description, xacro)
@@ -56,14 +56,6 @@
   </joint>
   <!-- Touch haptic devices -->
-  <xacro:property name="touch_descr" value="$(find touch_description)/urdf/touch.urdf.xacro" />
-  <xacro:if value="${len(touch_descr) == 0}">
-    <link name="touch_left_base" />
-    <link name="touch_right_base" />
-  </xacro:if>
-  <xacro:unless value="${len(touch_descr) == 0}">
-    <xacro:include filename="${touch_descr}" />
-    <xacro:touch prefix="touch_left_" />
-    <xacro:touch prefix="touch_right_" />
-  </xacro:unless>
+  <link name="touch_left_base" />
+  <link name="touch_right_base" />
   <joint name="world_touch_left_fixed" type="fixed">
     <parent link="world" />

Commit message: description: Swap tool(adapter)s

File: ursurg_description/urdf/ursurg.urdf.xacro (robot description, xacro)
@@ -14,11 +14,11 @@
     <origin xyz="0.6 -0.2 0" rpy="0 0 ${pi/2}" />
   </joint>
-  <!-- A) LND 420006 tool -->
-  <xacro:lnd420006 prefix="a_tool_" />
+  <!-- A) LND 470006 tool -->
+  <xacro:lnd470006 prefix="a_tool_" />
   <joint name="a_ur_tool_joint" type="fixed">
     <parent link="a_ur_ee_link" />
     <child link="a_tool_mount" />
     <!-- TODO: Calibrate to find this transform accurately -->
-    <origin xyz="0.075 0 -0.04" rpy="${pi} 0 0" />
+    <origin xyz="0.09 0 0" rpy="${pi} 0 0" />
   </joint>
   <!-- B) UR5 robot -->
@@ -31,11 +31,11 @@
     <origin xyz="0.6 -1 0" rpy="0 0 ${pi/2}" />
   </joint>
-  <!-- B) LND 470006 tool -->
-  <xacro:lnd470006 prefix="b_tool_" />
+  <!-- B) LND 420006 tool -->
+  <xacro:lnd420006 prefix="b_tool_" />
   <joint name="b_eua2_tool_joint" type="fixed">
     <parent link="b_ur_ee_link" />
     <child link="b_tool_mount" />
     <!-- TODO: Calibrate to find this transform accurately -->
-    <origin xyz="0.09 0 0" rpy="${pi} 0 0" />
+    <origin xyz="0.075 0 -0.04" rpy="${pi} 0 0" />
   </joint>
   <!-- Table -->

Commit message: ursurg_description: Update URDF to match current lab configuration

File: ursurg_description/urdf/ursurg.urdf.xacro (robot description, xacro)
@@ -12,5 +12,5 @@
     <parent link="world" />
     <child link="a_ur_base_link" />
-    <origin xyz="0.6 -0.2 0" rpy="0 0 ${pi/2}" />
+    <origin xyz="0 0.4 0" rpy="0 0 ${pi/2}" />
   </joint>
   <!-- A) LND 470006 tool -->
@@ -29,5 +29,5 @@
     <parent link="world" />
     <child link="b_ur_base_link" />
-    <origin xyz="0.6 -1 0" rpy="0 0 ${pi/2}" />
+    <origin xyz="0 -0.4 0" rpy="0 0 ${pi/2}" />
   </joint>
   <!-- B) LND 420006 tool -->
@@ -37,21 +37,5 @@
     <child link="b_tool_mount" />
     <!-- TODO: Calibrate to find this transform accurately -->
-    <origin xyz="0.075 0 -0.04" rpy="${pi} 0 0" />
-  </joint>
-  <!-- Table -->
-  <link name="table_base">
-    <visual>
-      <origin xyz="0.4 -0.6 -0.4" rpy="0 0 ${pi/2}" />
-      <geometry>
-        <box size="1.2 0.8 0.8" />
-      </geometry>
-      <material name="table_color">
-        <color rgba="0.55 0.45 0.3 1.0" />
-      </material>
-    </visual>
-  </link>
-  <joint name="world_table_base_joint" type="fixed">
-    <parent link="world" />
-    <child link="table_base" />
+    <origin xyz="0.075 0 0.04" rpy="0 0 0" />
   </joint>
   <!-- Touch haptic devices -->
@@ -68,3 +52,37 @@
     <origin xyz="-0.6 -0.7 0" rpy="0 0 ${pi/2}" />
   </joint>
+  <!-- Robot platform -->
+  <link name="platform">
+    <visual>
+      <origin xyz="0 0 -0.4" rpy="0 0 ${pi/2}" />
+      <geometry>
+        <box size="1.2 0.8 0.8" />
+      </geometry>
+      <material name="platform_color">
+        <color rgba="0.55 0.45 0.3 1.0" />
+      </material>
+    </visual>
+  </link>
+  <joint name="world_platform_joint" type="fixed">
+    <parent link="world" />
+    <child link="platform" />
+    <origin xyz="-0.2 0 0" rpy="0 0 0" />
+  </joint>
+  <!-- Operating table -->
+  <link name="operating_table">
+    <visual>
+      <origin xyz="0 0 -0.245" rpy="0 0 ${pi/2}" />
+      <geometry>
+        <box size="0.635 0.49 0.49" />
+      </geometry>
+      <material name="operating_table_color">
+        <color rgba="0.55 0.45 0.3 1.0" />
+      </material>
+    </visual>
+  </link>
+  <joint name="world_operating_table_joint" type="fixed">
+    <parent link="world" />
+    <child link="operating_table" />
+    <origin xyz="0.5 0 -0.31" rpy="0 0 0" />
+  </joint>
 </robot>

Commit message: description: Fix scene measurements

File: ursurg_description/urdf/ursurg.urdf.xacro (robot description, xacro)
@@ -55,7 +55,7 @@
   <link name="platform">
     <visual>
-      <origin xyz="0 0 -0.4" rpy="0 0 ${pi/2}" />
+      <origin xyz="0 0 ${-0.815/2}" rpy="0 0 ${pi/2}" />
       <geometry>
-        <box size="1.2 0.8 0.8" />
+        <box size="1.2 0.8 0.815" />
       </geometry>
       <material name="platform_color">
@@ -72,7 +72,7 @@
   <link name="operating_table">
     <visual>
-      <origin xyz="0 0 -0.245" rpy="0 0 ${pi/2}" />
+      <origin xyz="0 0 ${-0.55/2}" rpy="0 0 ${pi/2}" />
       <geometry>
-        <box size="0.635 0.49 0.49" />
+        <box size="0.635 0.49 0.55" />
       </geometry>
       <material name="operating_table_color">

Commit message: Added proper transformation for haptic devices

File: ursurg_description/urdf/ursurg.urdf.xacro (robot description, xacro)
@@ -42,10 +42,10 @@
     <parent link="world" />
     <child link="touch_left_base" />
-    <origin xyz="-0.6 -0.5 0" rpy="0 0 ${pi/2}" />
+    <origin xyz="0.3 -1.0 0" rpy="${pi/2} 0 0" />
   </joint>
   <joint name="world_touch_right_fixed" type="fixed">
     <parent link="world" />
     <child link="touch_right_base" />
-    <origin xyz="-0.6 -0.7 0" rpy="0 0 ${pi/2}" />
+    <origin xyz="0.6 -1.0 0" rpy="${pi/2} 0 0" />
   </joint>
   <!-- Robot platform -->

Commit message: description: Add calibration for robot A

File: ursurg_description/urdf/ursurg.urdf.xacro (robot description, xacro)
@@ -18,6 +18,5 @@
     <parent link="a_ur_ee_link" />
     <child link="a_tool_tip_calib" />
-    <!-- TODO: Calibrate to find this transform accurately -->
-    <origin xyz="0.66 0 0" rpy="0 0 0" />
+    <origin xyz="0.6634 -0.00077763 0.0078248" rpy="0 0 0" /> <!-- From calibration -->
   </joint>
   <!-- B) UR5 robot -->

Commit message: description: Place haptic device origin in front of robots

File: ursurg_description/urdf/ursurg.urdf.xacro (robot description, xacro)
@@ -55,10 +55,10 @@
     <parent link="world" />
     <child link="touch_left_base" />
-    <origin xyz="0.3 -1.0 0" rpy="${pi/2} 0 0" />
+    <origin xyz="0.5 -0.1 0.2" rpy="${pi/2} 0 ${pi/2}" />
   </joint>
   <joint name="world_touch_right_fixed" type="fixed">
     <parent link="world" />
     <child link="touch_right_base" />
-    <origin xyz="0.6 -1.0 0" rpy="${pi/2} 0 0" />
+    <origin xyz="0.5 0.1 0.2" rpy="${pi/2} 0 ${pi/2}" />
   </joint>
   <!-- Robot platform -->

Commit message: description: Move haptics devices origin further away from robots

File: ursurg_description/urdf/ursurg.urdf.xacro (robot description, xacro)
@@ -55,10 +55,10 @@
     <parent link="world" />
     <child link="touch_left_base" />
-    <origin xyz="0.5 -0.1 0.2" rpy="${pi/2} 0 ${pi/2}" />
+    <origin xyz="1 -0.1 0" rpy="${pi/2} 0 ${pi/2}" />
   </joint>
   <joint name="world_touch_right_fixed" type="fixed">
     <parent link="world" />
     <child link="touch_right_base" />
-    <origin xyz="0.5 0.1 0.2" rpy="${pi/2} 0 ${pi/2}" />
+    <origin xyz="1 0.1 0" rpy="${pi/2} 0 ${pi/2}" />
   </joint>
   <!-- Robot platform -->

Commit message: description: Update tool A calibration

File: ursurg_description/urdf/ursurg.urdf.xacro (robot description, xacro)
@@ -25,5 +25,5 @@
     <parent link="a_ur_ee_link" />
     <child link="a_tool_tip_calib" />
-    <origin xyz="0.6634 -0.00077763 0.0078248" rpy="0 0 0" /> <!-- From calibration -->
+    <origin xyz="0.64045, 0.0021887, 0.035773" rpy="0 0 0" /> <!-- From calibration -->
   </joint>
   <!-- B) UR5 robot -->

Commit message: description: Fix comma in values

File: ursurg_description/urdf/ursurg.urdf.xacro (robot description, xacro)
@@ -25,5 +25,5 @@
     <parent link="a_ur_ee_link" />
     <child link="a_tool_tip_calib" />
-    <origin xyz="0.64045, 0.0021887, 0.035773" rpy="0 0 0" /> <!-- From calibration -->
+    <origin xyz="0.64045 0.0021887 0.035773" rpy="0 0 0" /> <!-- From calibration -->
   </joint>
   <!-- B) UR5 robot -->

Commit message: description: Remove operating table object

File: ursurg_description/urdf/ursurg.urdf.xacro (robot description, xacro)
@@ -79,20 +79,3 @@
     <origin xyz="-0.2 0 0" rpy="0 0 0" />
   </joint>
-  <!-- Operating table -->
-  <link name="operating_table">
-    <visual>
-      <origin xyz="0 0 ${-0.55/2}" rpy="0 0 ${pi/2}" />
-      <geometry>
-        <box size="0.635 0.49 0.55" />
-      </geometry>
-      <material name="operating_table_color">
-        <color rgba="0.55 0.45 0.3 1.0" />
-      </material>
-    </visual>
-  </link>
-  <joint name="world_operating_table_joint" type="fixed">
-    <parent link="world" />
-    <child link="operating_table" />
-    <origin xyz="0.5 0 -0.31" rpy="0 0 0" />
-  </joint>
 </robot>

Commit message: description: Align Touch devices to camera frame

File: ursurg_description/urdf/ursurg.urdf.xacro (robot description, xacro)
@@ -53,12 +53,12 @@
   <link name="touch_right_base" />
   <joint name="world_touch_left_fixed" type="fixed">
-    <parent link="world" />
+    <parent link="stereo_optical" />
     <child link="touch_left_base" />
-    <origin xyz="1 -0.1 0" rpy="${pi/2} 0 ${pi/2}" />
+    <origin xyz="-0.15 0 0" rpy="0 ${pi} ${pi}" />
   </joint>
   <joint name="world_touch_right_fixed" type="fixed">
-    <parent link="world" />
+    <parent link="stereo_optical" />
     <child link="touch_right_base" />
-    <origin xyz="1 0.1 0" rpy="${pi/2} 0 ${pi/2}" />
+    <origin xyz="0.15 0 0" rpy="0 ${pi} ${pi}" />
   </joint>
   <!-- Robot platform -->

Commit message: description: Add uncalibrated camera frame

File: ursurg_description/urdf/ursurg.urdf.xacro (robot description, xacro)
@@ -49,4 +49,11 @@
     <origin xyz="0.56961 -0.0012618 0.056071" rpy="0 0 0" /> <!-- From calibration -->
   </joint>
+  <!-- Stereo camera -->
+  <link name="stereo_optical" />
+  <joint name="world_stereo_optical_fixed" type="fixed">
+    <parent link="world" />
+    <child link="stereo_optical" />
+    <origin xyz="0.2 0 0.1" rpy="${-3*pi/4} 0 ${-pi/2}" />
+  </joint>
   <!-- Touch haptic devices -->
   <link name="touch_left_base" />

Commit message: description: Remove platform visuals

File: ursurg_description/urdf/ursurg.urdf.xacro (robot description, xacro)
@@ -69,20 +69,3 @@
     <origin xyz="0.15 0 0" rpy="0 ${pi} ${pi}" />
   </joint>
-  <!-- Robot platform -->
-  <link name="platform">
-    <visual>
-      <origin xyz="0 0 ${-0.815/2}" rpy="0 0 ${pi/2}" />
-      <geometry>
-        <box size="1.2 0.8 0.815" />
-      </geometry>
-      <material name="platform_color">
-        <color rgba="0.55 0.45 0.3 1.0" />
-      </material>
-    </visual>
-  </link>
-  <joint name="world_platform_joint" type="fixed">
-    <parent link="world" />
-    <child link="platform" />
-    <origin xyz="-0.2 0 0" rpy="0 0 0" />
-  </joint>
 </robot>

Commit message: Add new tool calibration

File: ursurg_description/urdf/ursurg.urdf.xacro (robot description, xacro)
@@ -3,7 +3,5 @@
   <xacro:include filename="lnd.urdf.xacro" />
   <link name="world" />
-  <!-- A) UR5e robot
-       Run xacro with arg 'kinematics_config_file' set to override the default
-       kinematic configuration -->
+  <!-- A) UR5e robot -->
   <xacro:include filename="$(find ur_e_description)/urdf/ur5e.urdf.xacro" />
   <xacro:ur5e_robot prefix="a_ur_" joint_limited="true"
@@ -22,8 +20,10 @@
   <!-- A) LND 470006 tool -->
   <xacro:lnd470006 prefix="a_tool_" />
+  <xacro:property name="a_tool_calib_data" value="${load_yaml('$(arg a_tool_calib_file)')}" />
+  <xacro:property name="a_tcp_offset" value="${a_tool_calib_data['tcp_offset']}" />
   <joint name="a_ur_tool_joint" type="fixed">
     <parent link="a_ur_ee_link" />
     <child link="a_tool_tip_calib" />
-    <origin xyz="0.64045 0.0021887 0.035773" rpy="0 0 0" /> <!-- From calibration -->
+    <origin xyz="${a_tcp_offset['x']} ${a_tcp_offset['y']} ${a_tcp_offset['z']}" rpy="0 0 0" /> <!-- From calibration -->
   </joint>
   <!-- B) UR5 robot -->
@@ -44,8 +44,10 @@
   <!-- B) LND 420006 tool -->
   <xacro:lnd420006 prefix="b_tool_" />
+  <xacro:property name="b_tool_calib_data" value="${load_yaml('$(arg b_tool_calib_file)')}" />
+  <xacro:property name="b_tcp_offset" value="${b_tool_calib_data['tcp_offset']}" />
   <joint name="b_eua2_tool_joint" type="fixed">
     <parent link="b_ur_ee_link" />
     <child link="b_tool_tip_calib" />
-    <origin xyz="0.56961 -0.0012618 0.056071" rpy="0 0 0" /> <!-- From calibration -->
+    <origin xyz="${b_tcp_offset['x']} ${b_tcp_offset['y']} ${b_tcp_offset['z']}" rpy="0 0 0" />
   </joint>
   <!-- Stereo camera -->

Commit message: description: Change yaml format

File: ursurg_description/urdf/ursurg.urdf.xacro (robot description, xacro)
@@ -21,9 +21,9 @@
   <xacro:lnd470006 prefix="a_tool_" />
   <xacro:property name="a_tool_calib_data" value="${load_yaml('$(arg a_tool_calib_file)')}" />
-  <xacro:property name="a_tcp_offset" value="${a_tool_calib_data['tcp_offset']}" />
+  <xacro:property name="a_robot_to_tool" value="${a_tool_calib_data['robot_to_tool']}" />
   <joint name="a_ur_tool_joint" type="fixed">
     <parent link="a_ur_ee_link" />
     <child link="a_tool_tip_calib" />
-    <origin xyz="${a_tcp_offset['x']} ${a_tcp_offset['y']} ${a_tcp_offset['z']}" rpy="0 0 0" /> <!-- From calibration -->
+    <origin xyz="${' '.join(str(val) for val in a_robot_to_tool['xyz'])}" rpy="${' '.join(str(val) for val in a_robot_to_tool['rpy'])}" />
   </joint>
   <!-- B) UR5 robot -->
@@ -45,9 +45,9 @@
   <xacro:lnd420006 prefix="b_tool_" />
   <xacro:property name="b_tool_calib_data" value="${load_yaml('$(arg b_tool_calib_file)')}" />
-  <xacro:property name="b_tcp_offset" value="${b_tool_calib_data['tcp_offset']}" />
+  <xacro:property name="b_robot_to_tool" value="${b_tool_calib_data['robot_to_tool']}" />
   <joint name="b_eua2_tool_joint" type="fixed">
     <parent link="b_ur_ee_link" />
     <child link="b_tool_tip_calib" />
-    <origin xyz="${b_tcp_offset['x']} ${b_tcp_offset['y']} ${b_tcp_offset['z']}" rpy="0 0 0" />
+    <origin xyz="${' '.join(str(val) for val in b_robot_to_tool['xyz'])}" rpy="${' '.join(str(val) for val in b_robot_to_tool['rpy'])}" />
   </joint>
   <!-- Stereo camera -->

Commit message: description: Add world calibration YAML file

File: ursurg_description/urdf/ursurg.urdf.xacro (robot description, xacro)
@@ -3,4 +3,6 @@
   <xacro:include filename="lnd.urdf.xacro" />
   <link name="world" />
+  <xacro:property name="world_calib_file" value="$(find ursurg_description)/config/world_calib.yaml" />
+  <xacro:property name="world_calib_data" value="${load_yaml(world_calib_file)}" />
   <!-- A) UR5e robot -->
   <xacro:include filename="$(find ur_e_description)/urdf/ur5e.urdf.xacro" />
@@ -13,8 +15,10 @@
     wrist_3_lower_limit="${-pi}" wrist_3_upper_limit="${pi}"
     kinematics_file="${load_yaml('$(arg a_kinematics_config_file)')}" />
+  <xacro:property name="world_to_a_base_link" value="${world_calib_data['world_to_a_base_link']}" />
   <joint name="a_world_ur_base_joint" type="fixed">
     <parent link="world" />
     <child link="a_ur_base_link" />
-    <origin xyz="0 0.4 0" rpy="0 0 ${pi/2}" />
+    <origin xyz="${' '.join(str(val) for val in world_to_a_base_link['xyz'])}"
+      rpy="${' '.join(str(val) for val in world_to_a_base_link['rpy'])}" />
   </joint>
   <!-- A) LND 470006 tool -->
@@ -25,5 +29,6 @@
     <parent link="a_ur_ee_link" />
     <child link="a_tool_tip_calib" />
-    <origin xyz="${' '.join(str(val) for val in a_robot_to_tool['xyz'])}" rpy="${' '.join(str(val) for val in a_robot_to_tool['rpy'])}" />
+    <origin xyz="${' '.join(str(val) for val in a_robot_to_tool['xyz'])}"
+      rpy="${' '.join(str(val) for val in a_robot_to_tool['rpy'])}" />
   </joint>
   <!-- B) UR5 robot -->
@@ -37,8 +42,10 @@
     wrist_3_lower_limit="${-pi}" wrist_3_upper_limit="${pi}"
     kinematics_file="${load_yaml('$(arg b_kinematics_config_file)')}" />
+  <xacro:property name="world_to_b_base_link" value="${world_calib_data['world_to_b_base_link']}" />
   <joint name="b_world_ur_base_joint" type="fixed">
     <parent link="world" />
     <child link="b_ur_base_link" />
-    <origin xyz="0 -0.4 0" rpy="0 0 ${pi/2}" />
+    <origin xyz="${' '.join(str(val) for val in world_to_b_base_link['xyz'])}"
+      rpy="${' '.join(str(val) for val in world_to_b_base_link['rpy'])}" />
   </joint>
   <!-- B) LND 420006 tool -->
@@ -49,12 +56,15 @@
     <parent link="b_ur_ee_link" />
     <child link="b_tool_tip_calib" />
-    <origin xyz="${' '.join(str(val) for val in b_robot_to_tool['xyz'])}" rpy="${' '.join(str(val) for val in b_robot_to_tool['rpy'])}" />
+    <origin xyz="${' '.join(str(val) for val in b_robot_to_tool['xyz'])}"
+      rpy="${' '.join(str(val) for val in b_robot_to_tool['rpy'])}" />
   </joint>
   <!-- Stereo camera -->
   <link name="stereo_optical" />
+  <xacro:property name="world_to_stereo_optical" value="${world_calib_data['world_to_stereo_optical']}" />
   <joint name="world_stereo_optical_fixed" type="fixed">
     <parent link="world" />
     <child link="stereo_optical" />
-    <origin xyz="0.2 0 0.1" rpy="${-3*pi/4} 0 ${-pi/2}" />
+    <origin xyz="${' '.join(str(val) for val in world_to_stereo_optical['xyz'])}"
+      rpy="${' '.join(str(val) for val in world_to_stereo_optical['rpy'])}" />
   </joint>
   <!-- Touch haptic devices -->
