Commit message: description: Define haptic device base wrt. robot base

File: ursurg_description/urdf/ursurg.urdf.xacro (robot description, xacro)
@@ -72,12 +72,12 @@
   <link name="touch_right_base" />
   <joint name="world_touch_left_fixed" type="fixed">
-    <parent link="stereo_optical" />
+    <parent link="a_ur_base_link" />
     <child link="touch_left_base" />
-    <origin xyz="-0.15 0 0" rpy="0 ${pi} ${pi}" />
+    <origin xyz="-0.3 -0.4 0.1" rpy="${pi/2} 0 ${pi}" />
   </joint>
   <joint name="world_touch_right_fixed" type="fixed">
-    <parent link="stereo_optical" />
+    <parent link="b_ur_base_link" />
     <child link="touch_right_base" />
-    <origin xyz="0.15 0 0" rpy="0 ${pi} ${pi}" />
+    <origin xyz="0.3 -0.4 0.1" rpy="${pi/2} 0 ${pi}" />
   </joint>
 </robot>

Commit message: description: Update UR base link frame name

File: ursurg_description/urdf/ursurg.urdf.xacro (robot description, xacro)
@@ -22,5 +22,5 @@
   <xacro:property name="a_robot_to_tool" value="${a_tool_calib_data['robot_to_tool']}" />
   <joint name="a_ur_tool_joint" type="fixed">
-    <parent link="a_ur_ee_link" />
+    <parent link="a_ur_flange" />
     <child link="a_tool_tip_calib" />
     <origin xyz="${' '.join(str(val) for val in a_robot_to_tool['xyz'])}"
@@ -44,5 +44,5 @@
   <xacro:property name="b_robot_to_tool" value="${b_tool_calib_data['robot_to_tool']}" />
   <joint name="b_eua2_tool_joint" type="fixed">
-    <parent link="b_ur_ee_link" />
+    <parent link="b_ur_flange" />
     <child link="b_tool_tip_calib" />
     <origin xyz="${' '.join(str(val) for val in b_robot_to_tool['xyz'])}"
