Commit message: description: Convert to ROS2

File: mops_description/urdf/mops.urdf.xacro (robot description, xacro)
@@ -2,19 +2,27 @@
 <robot name="ursurg" xmlns:xacro="http://ros.org/wiki/xacro">
   <xacro:include filename="lnd.urdf.xacro" />
+  <xacro:include filename="$(find ur_description)/urdf/ur_macro.xacro" />
   <link name="world" />
-  <xacro:property name="world_calib_file" value="$(find ursurg_description)/config/world_calib.yaml" />
+  <xacro:property name="world_calib_file" value="$(find mops_description)/config/world_calib.yaml" />
   <xacro:property name="world_calib_data" value="${load_yaml(world_calib_file)}" />
   <!-- A) UR5e robot -->
-  <xacro:include filename="$(find ur_description)/urdf/inc/ur5e_macro.xacro" />
-  <xacro:ur5e_robot
-    prefix="a_ur_"
-    kinematics_parameters_file="$(arg a_kinematics_config_file)" />
   <xacro:property name="world_to_a_base_link" value="${world_calib_data['world_to_a_base_link']}" />
-  <joint name="a_world_ur_base_joint" type="fixed">
+  <xacro:ur_robot
+      name="ur_a"
+      prefix="a_ur_"
+      parent="world"
+      joint_limits_parameters_file="$(find ur_description)/config/ur5e/joint_limits.yaml"
+      kinematics_parameters_file="$(find ur_description)/config/ur5e/default_kinematics.yaml"
+      physical_parameters_file="$(find ur_description)/config/ur5e/physical_parameters.yaml"
+      visual_parameters_file="$(find ur_description)/config/ur5e/visual_parameters.yaml">
+    <origin xyz="${' '.join(str(val) for val in world_to_a_base_link['xyz'])}"
+        rpy="${' '.join(str(val) for val in world_to_a_base_link['rpy'])}" />
+  </xacro:ur_robot>
+  <!-- <joint name="a_world_ur_base_joint" type="fixed">
     <parent link="world" />
     <child link="a_ur_base_link" />
     <origin xyz="${' '.join(str(val) for val in world_to_a_base_link['xyz'])}"
       rpy="${' '.join(str(val) for val in world_to_a_base_link['rpy'])}" />
-  </joint>
+  </joint> -->
   <!-- A) LND 470006 tool -->
   <xacro:lnd470006 prefix="a_tool_" />
@@ -28,15 +36,22 @@
   </joint>
   <!-- B) UR5 robot -->
-  <xacro:include filename="$(find ur_description)/urdf/inc/ur5_macro.xacro" />
-  <xacro:ur5_robot
-    prefix="b_ur_"
-    kinematics_parameters_file="$(arg b_kinematics_config_file)" />
   <xacro:property name="world_to_b_base_link" value="${world_calib_data['world_to_b_base_link']}" />
-  <joint name="b_world_ur_base_joint" type="fixed">
+  <xacro:ur_robot
+      name="ur_b"
+      prefix="b_ur_"
+      parent="world"
+      joint_limit_params_file="$(find ur_description)/config/ur5/joint_limits.yaml"
+      kinematics_params_file="$(find ur_description)/config/ur5/default_kinematics.yaml"
+      physical_params_file="$(find ur_description)/config/ur5/physical_parameters.yaml"
+      visual_params_file="$(find ur_description)/config/ur5/visual_parameters.yaml">
+    <origin xyz="${' '.join(str(val) for val in world_to_b_base_link['xyz'])}"
+        rpy="${' '.join(str(val) for val in world_to_b_base_link['rpy'])}" />
+  </xacro:ur_robot>
+  <!-- <joint name="b_world_ur_base_joint" type="fixed">
     <parent link="world" />
     <child link="b_ur_base_link" />
     <origin xyz="${' '.join(str(val) for val in world_to_b_base_link['xyz'])}"
       rpy="${' '.join(str(val) for val in world_to_b_base_link['rpy'])}" />
-  </joint>
+  </joint> -->
   <!-- B) LND 420006 tool -->
   <xacro:lnd420006 prefix="b_tool_" />

Commit message: description: Fix use official ur_description

File: mops_description/urdf/mops.urdf.xacro (robot description, xacro)
@@ -1,9 +1,17 @@
 <?xml version="1.0"?>
-<robot name="ursurg" xmlns:xacro="http://ros.org/wiki/xacro">
+<robot name="mops" xmlns:xacro="http://ros.org/wiki/xacro">
+  <xacro:include filename="$(find ur_description)/urdf/ur_macro.xacro" />
   <xacro:include filename="lnd.urdf.xacro" />
-  <xacro:include filename="$(find ur_description)/urdf/ur_macro.xacro" />
-  <link name="world" />
+  <xacro:arg name="a_joint_limit_params_file" default="$(find ur_description)/config/ur5e/joint_limits.yaml"/>
+  <xacro:arg name="a_kinematics_params_file" default="$(find ur_description)/config/ur5e/default_kinematics.yaml"/>
+  <xacro:arg name="a_physical_params_file" default="$(find ur_description)/config/ur5e/physical_parameters.yaml"/>
+  <xacro:arg name="a_visual_params_file" default="$(find ur_description)/config/ur5e/visual_parameters.yaml"/>
+  <xacro:arg name="b_joint_limit_params_file" default="$(find ur_description)/config/ur5/joint_limits.yaml"/>
+  <xacro:arg name="b_kinematics_params_file" default="$(find ur_description)/config/ur5/default_kinematics.yaml"/>
+  <xacro:arg name="b_physical_params_file" default="$(find ur_description)/config/ur5/physical_parameters.yaml"/>
+  <xacro:arg name="b_visual_params_file" default="$(find ur_description)/config/ur5/visual_parameters.yaml"/>
   <xacro:property name="world_calib_file" value="$(find mops_description)/config/world_calib.yaml" />
   <xacro:property name="world_calib_data" value="${load_yaml(world_calib_file)}" />
+  <link name="world" />
   <!-- A) UR5e robot -->
   <xacro:property name="world_to_a_base_link" value="${world_calib_data['world_to_a_base_link']}" />
@@ -12,8 +20,9 @@
       prefix="a_ur_"
       parent="world"
-      joint_limits_parameters_file="$(find ur_description)/config/ur5e/joint_limits.yaml"
-      kinematics_parameters_file="$(find ur_description)/config/ur5e/default_kinematics.yaml"
-      physical_parameters_file="$(find ur_description)/config/ur5e/physical_parameters.yaml"
-      visual_parameters_file="$(find ur_description)/config/ur5e/visual_parameters.yaml">
+      joint_limits_parameters_file="$(arg a_joint_limit_params_file)"
+      kinematics_parameters_file="$(arg a_kinematics_params_file)"
+      physical_parameters_file="$(arg a_physical_params_file)"
+      visual_parameters_file="$(arg a_visual_params_file)"
+      transmission_hw_interface="">
     <origin xyz="${' '.join(str(val) for val in world_to_a_base_link['xyz'])}"
         rpy="${' '.join(str(val) for val in world_to_a_base_link['rpy'])}" />
@@ -41,8 +50,9 @@
       prefix="b_ur_"
       parent="world"
-      joint_limit_params_file="$(find ur_description)/config/ur5/joint_limits.yaml"
-      kinematics_params_file="$(find ur_description)/config/ur5/default_kinematics.yaml"
-      physical_params_file="$(find ur_description)/config/ur5/physical_parameters.yaml"
-      visual_params_file="$(find ur_description)/config/ur5/visual_parameters.yaml">
+      joint_limits_parameters_file="$(arg b_joint_limit_params_file)"
+      kinematics_parameters_file="$(arg b_kinematics_params_file)"
+      physical_parameters_file="$(arg b_physical_params_file)"
+      visual_parameters_file="$(arg b_visual_params_file)"
+      transmission_hw_interface="">
     <origin xyz="${' '.join(str(val) for val in world_to_b_base_link['xyz'])}"
         rpy="${' '.join(str(val) for val in world_to_b_base_link['rpy'])}" />

Commit message: description: Quick fix to rotate tools on UR flange
Something seems to have changed in the official ur_description model.

File: mops_description/urdf/mops.urdf.xacro (robot description, xacro)
@@ -34,6 +34,13 @@
   <xacro:property name="a_tool_calib_data" value="${load_yaml(a_tool_calib_file_prop)}" />
   <xacro:property name="a_robot_to_tool" value="${a_tool_calib_data['robot_to_tool']}" />
+  <!-- FIXME remove this intermediate link -->
+  <link name="a_flange_tool_fix" />
+  <joint name="a_ur_tool_joint_fix" type="fixed">
+    <parent link="a_ur_flange" />
+    <child link="a_flange_tool_fix" />
+    <origin xyz="0 0 0" rpy="${pi} 0 0" />
+  </joint>
   <joint name="a_ur_tool_joint" type="fixed">
-    <parent link="a_ur_flange" />
+    <parent link="a_flange_tool_fix" />
     <child link="a_tool_tip_calib" />
     <origin xyz="${' '.join(str(val) for val in a_robot_to_tool['xyz'])}"
@@ -59,6 +66,13 @@
   <xacro:property name="b_tool_calib_data" value="${load_yaml(b_tool_calib_file_prop)}" />
   <xacro:property name="b_robot_to_tool" value="${b_tool_calib_data['robot_to_tool']}" />
-  <joint name="b_eua2_tool_joint" type="fixed">
+  <!-- FIXME remove this intermediate link -->
+  <link name="b_flange_tool_fix" />
+  <joint name="b_ur_tool_joint_fix" type="fixed">
     <parent link="b_ur_flange" />
+    <child link="b_flange_tool_fix" />
+    <origin xyz="0 0 0" rpy="${pi} 0 0" />
+  </joint>
+  <joint name="b_ur_tool_joint" type="fixed">
+    <parent link="b_flange_tool_fix" />
     <child link="b_tool_tip_calib" />
     <origin xyz="${' '.join(str(val) for val in b_robot_to_tool['xyz'])}"

Commit message: description: Update tool models
Do not rely on old calibration parameters.

File: mops_description/urdf/mops.urdf.xacro (robot description, xacro)
@@ -1,14 +1,14 @@
 <?xml version="1.0"?>
 <robot name="mops" xmlns:xacro="http://ros.org/wiki/xacro">
-  <xacro:include filename="$(find ur_description)/urdf/ur_macro.xacro" />
-  <xacro:include filename="lnd.urdf.xacro" />
-  <xacro:arg name="a_joint_limit_params_file" default="$(find ur_description)/config/ur5e/joint_limits.yaml"/>
-  <xacro:arg name="a_kinematics_params_file" default="$(find ur_description)/config/ur5e/default_kinematics.yaml"/>
-  <xacro:arg name="a_physical_params_file" default="$(find ur_description)/config/ur5e/physical_parameters.yaml"/>
-  <xacro:arg name="a_visual_params_file" default="$(find ur_description)/config/ur5e/visual_parameters.yaml"/>
-  <xacro:arg name="b_joint_limit_params_file" default="$(find ur_description)/config/ur5/joint_limits.yaml"/>
-  <xacro:arg name="b_kinematics_params_file" default="$(find ur_description)/config/ur5/default_kinematics.yaml"/>
-  <xacro:arg name="b_physical_params_file" default="$(find ur_description)/config/ur5/physical_parameters.yaml"/>
-  <xacro:arg name="b_visual_params_file" default="$(find ur_description)/config/ur5/visual_parameters.yaml"/>
+  <xacro:include filename="$(find ur_description)/urdf/ur_macro.xacro" /> <!-- From 'ros-humble-ur-description' -->
+  <xacro:include filename="$(find mops_description)/urdf/dv_tools.urdf.xacro" />
+  <xacro:arg name="a_joint_limit_params_file" default="$(find ur_description)/config/ur5e/joint_limits.yaml" />
+  <xacro:arg name="a_kinematics_params_file" default="$(find ur_description)/config/ur5e/default_kinematics.yaml" />
+  <xacro:arg name="a_physical_params_file" default="$(find ur_description)/config/ur5e/physical_parameters.yaml" />
+  <xacro:arg name="a_visual_params_file" default="$(find ur_description)/config/ur5e/visual_parameters.yaml" />
+  <xacro:arg name="b_joint_limit_params_file" default="$(find ur_description)/config/ur5/joint_limits.yaml" />
+  <xacro:arg name="b_kinematics_params_file" default="$(find ur_description)/config/ur5/default_kinematics.yaml" />
+  <xacro:arg name="b_physical_params_file" default="$(find ur_description)/config/ur5/physical_parameters.yaml" />
+  <xacro:arg name="b_visual_params_file" default="$(find ur_description)/config/ur5/visual_parameters.yaml" />
   <!-- <xacro:arg name="world_calib_file" default="" /> -->
   <xacro:property name="world_calib_file_prop" value="$(arg world_calib_file)" />
@@ -30,21 +30,7 @@
   </xacro:ur_robot>
   <!-- A) LND 470006 tool -->
-  <xacro:lnd470006 prefix="a_tool_" />
-  <xacro:property name="a_tool_calib_file_prop" value="$(arg a_tool_calib_file)" />
-  <xacro:property name="a_tool_calib_data" value="${load_yaml(a_tool_calib_file_prop)}" />
-  <xacro:property name="a_robot_to_tool" value="${a_tool_calib_data['robot_to_tool']}" />
-  <!-- FIXME remove this intermediate link -->
-  <link name="a_flange_tool_fix" />
-  <joint name="a_ur_tool_joint_fix" type="fixed">
-    <parent link="a_ur_flange" />
-    <child link="a_flange_tool_fix" />
-    <origin xyz="0 0 0" rpy="${pi} 0 0" />
-  </joint>
-  <joint name="a_ur_tool_joint" type="fixed">
-    <parent link="a_flange_tool_fix" />
-    <child link="a_tool_tip_calib" />
-    <origin xyz="${' '.join(str(val) for val in a_robot_to_tool['xyz'])}"
-      rpy="${' '.join(str(val) for val in a_robot_to_tool['rpy'])}" />
-  </joint>
+  <xacro:dv_large_needle_driver_470006 prefix="a_tool_" parent="a_ur_flange">
+    <origin xyz="0.098 0 -0.053" rpy="0 ${pi/2} 0" /> <!-- FIXME -->
+  </xacro:dv_large_needle_driver_470006>
   <!-- B) UR5 robot -->
   <xacro:property name="world_to_b_base_link" value="${world_calib_data['world_to_b_base_link']}" />
@@ -62,30 +48,7 @@
   </xacro:ur_robot>
   <!-- B) LND 420006 tool -->
-  <xacro:lnd420006 prefix="b_tool_" />
-  <xacro:property name="b_tool_calib_file_prop" value="$(arg b_tool_calib_file)" />
-  <xacro:property name="b_tool_calib_data" value="${load_yaml(b_tool_calib_file_prop)}" />
-  <xacro:property name="b_robot_to_tool" value="${b_tool_calib_data['robot_to_tool']}" />
-  <!-- FIXME remove this intermediate link -->
-  <link name="b_flange_tool_fix" />
-  <joint name="b_ur_tool_joint_fix" type="fixed">
-    <parent link="b_ur_flange" />
-    <child link="b_flange_tool_fix" />
-    <origin xyz="0 0 0" rpy="${pi} 0 0" />
-  </joint>
-  <joint name="b_ur_tool_joint" type="fixed">
-    <parent link="b_flange_tool_fix" />
-    <child link="b_tool_tip_calib" />
-    <origin xyz="${' '.join(str(val) for val in b_robot_to_tool['xyz'])}"
-      rpy="${' '.join(str(val) for val in b_robot_to_tool['rpy'])}" />
-  </joint>
-  <!-- Stereo camera -->
-  <link name="stereo_optical" />
-  <xacro:property name="world_to_stereo_optical" value="${world_calib_data['world_to_stereo_optical']}" />
-  <joint name="world_stereo_optical_fixed" type="fixed">
-    <parent link="world" />
-    <child link="stereo_optical" />
-    <origin xyz="${' '.join(str(val) for val in world_to_stereo_optical['xyz'])}"
-      rpy="${' '.join(str(val) for val in world_to_stereo_optical['rpy'])}" />
-  </joint>
+  <xacro:dv_large_needle_driver_420006 prefix="b_tool_" parent="b_ur_flange">
+    <origin xyz="0.095 0 -0.053" rpy="0 0 0" /> <!-- FIXME -->
+  </xacro:dv_large_needle_driver_420006>
   <!-- Touch haptic devices -->
   <link name="touch_left_base" />

File: mops_description/urdf/tool/dv_large_needle_driver.urdf.xacro (robot description, xacro)
@@ -1,13 +1,7 @@
 <?xml version="1.0"?>
-<!-- da Vinci Large Needle Driver (LND) model 420006 (S/Si) and 470006 (X/Xi) -->
-<robot name="lnd" xmlns:xacro="http://ros.org/wiki/xacro">
-  <material name="tip_metallic_gray">
-    <color rgba="0.667 0.663 0.678 1.0" />
-  </material>
-  <material name="rod_dark_grey">
-    <color rgba="0.1 0.1 0.1 1.0" />
-  </material>
-  <xacro:macro name="lnd_tip" params="prefix" >
-    <link name="${prefix}tip_calib" />
+<!-- da Vinci Large Needle Driver (LND) models -->
+<robot name="dv_large_needle_driver" xmlns:xacro="http://ros.org/wiki/xacro">
+  <!-- End-effector of the LND -->
+  <xacro:macro name="dv_large_needle_driver_tip" params="prefix length" >
     <link name="${prefix}rotation">
       <visual>
@@ -52,7 +46,7 @@
     <link name="${prefix}tcp2" />
     <joint name="${prefix}roll" type="revolute">
-      <parent link="${prefix}tip_calib" />
+      <parent link="${prefix}base" />
       <child link="${prefix}rotation" />
-      <origin xyz="-0.018 0 0" rpy="${-pi} ${-pi/2} 0" />
+      <origin xyz="${length} 0 0" rpy="${-pi} ${-pi/2} 0" />
       <axis xyz="0 0 1" />
       <limit lower="${radians(-260)}" upper="${radians(260)}" effort="0.3" velocity="${2*pi}" />
@@ -71,5 +65,5 @@
     </joint>
     <!-- This is not a real physical joint, but rather yaw0 = (yaw1 - yaw2) / 2,
-         ie. the TCP frame is at an angle between the grasper jaws. -->
+          ie. the TCP frame is at an angle between the grasper jaws. -->
     <joint name="${prefix}yaw0" type="revolute">
       <parent link="${prefix}jaw_hinge" />
@@ -108,68 +102,74 @@
       <origin xyz="0.009 0 0" rpy="0 0 0" />
     </joint>
-  </xacro:macro>
-  <xacro:macro name="lnd420006" params="prefix">
-    <xacro:lnd_tip prefix="${prefix}" />
+  </xacro:macro> <!-- dv_large_needle_driver_tip -->
+  <!--  -->
+  <xacro:macro name="dv_large_needle_driver_housing_si" params="prefix" >
+    <link name="${prefix}housing">
+      <visual>
+        <geometry>
+          <box size="0.096 0.065 0.03" />
+        </geometry>
+        <material name="housing_light_blue" />
+      </visual>
+    </link>
+    <joint name="${prefix}housing_fixed" type="fixed">
+      <parent link="${prefix}base" />
+      <child link="${prefix}housing" />
+      <origin xyz="-0.025 0 0" rpy="0 0 0" /> <!-- FIXME -->
+    </joint>
+  </xacro:macro> <!-- dv_large_needle_driver_housing_si -->
+  <xacro:macro name="dv_large_needle_driver_housing_xi" params="prefix" >
+    <link name="${prefix}housing">
+      <visual>
+        <geometry>
+          <box size="0.06 0.045 0.08" />
+        </geometry>
+        <material name="housing_white" />
+      </visual>
+    </link>
+    <joint name="${prefix}housing_fixed" type="fixed">
+      <parent link="${prefix}base" />
+      <child link="${prefix}housing" />
+      <origin xyz="-0.015 0 -0.019" rpy="0 0 0" /> <!-- FIXME -->
+    </joint>
+  </xacro:macro> <!-- dv_large_needle_driver_housing_xi -->
+  <xacro:macro name="dv_large_needle_driver_rod" params="prefix length" >
     <link name="${prefix}rod">
       <visual>
         <geometry>
-          <cylinder radius="0.004" length="0.457" />
+          <cylinder radius="0.004" length="${length}" />
         </geometry>
         <material name="rod_dark_grey" />
       </visual>
     </link>
-    <joint name="${prefix}rod_joint" type="fixed">
+    <joint name="${prefix}rod_fixed" type="fixed">
       <parent link="${prefix}rotation" />
       <child link="${prefix}rod" />
-      <origin xyz="0 0 ${-0.457/2 - 0.01}" rpy="0 0 0" />
+      <origin xyz="0 0 ${-length/2 - 0.01}" rpy="0 0 0" />
     </joint>
-    <link name="${prefix}housing">
-      <visual>
-        <origin xyz="-0.013 0 0" rpy="0 0 0" />
-        <geometry>
-          <box size="0.096 0.065 0.03" />
-        </geometry>
-        <material name="housing_light_blue">
-          <color rgba="0.500 0.867 1.0 1.0" />
-        </material>
-      </visual>
-    </link>
-    <joint name="${prefix}housing_joint" type="fixed">
-      <parent link="${prefix}tip_calib" />
-      <child link="${prefix}housing" />
-      <origin xyz="${-0.018 - 0.01 - 0.457} 0 0" rpy="0 0 0" />
+  </xacro:macro> <!-- dv_large_needle_driver_rod -->
+  <xacro:macro name="dv_large_needle_driver_420006" params="prefix parent *origin">
+    <xacro:property name="length" value="0.4670" />
+    <link name="${prefix}base" />
+    <joint name="${prefix}base_fixed" type="fixed">
+      <xacro:insert_block name="origin" />
+      <parent link="${parent}" />
+      <child link="${prefix}base" />
     </joint>
-  </xacro:macro>
-  <xacro:macro name="lnd470006" params="prefix">
-    <xacro:lnd_tip prefix="${prefix}" />
-    <link name="${prefix}rod">
-      <visual>
-        <geometry>
-          <cylinder radius="0.004" length="0.5335" />
-        </geometry>
-        <material name="rod_dark_grey" />
-      </visual>
-    </link>
-    <joint name="${prefix}rod_joint" type="fixed">
-      <parent link="${prefix}rotation" />
-      <child link="${prefix}rod" />
-      <origin xyz="0 0 ${-0.5335/2 - 0.01}" rpy="0 0 0" />
+    <xacro:dv_large_needle_driver_tip prefix="${prefix}" length="${length}" />
+    <xacro:dv_large_needle_driver_rod prefix="${prefix}" length="${length}" />
+    <xacro:dv_large_needle_driver_housing_si prefix="${prefix}" />
+  </xacro:macro> <!-- dv_large_needle_driver_420006 -->
+  <xacro:macro name="dv_large_needle_driver_470006" params="prefix parent *origin">
+    <xacro:property name="length" value="0.5335" />
+    <link name="${prefix}base" />
+    <joint name="${prefix}base_fixed" type="fixed">
+      <xacro:insert_block name="origin" />
+      <parent link="${parent}" />
+      <child link="${prefix}base" />
     </joint>
-    <link name="${prefix}housing">
-      <visual>
-        <origin xyz="-0.015 0 -0.019" rpy="0 0 0" />
-        <geometry>
-          <box size="0.06 0.045 0.08" />
-        </geometry>
-        <material name="housing_white">
-          <color rgba="1.0 1.0 1.0 1.0" />
-        </material>
-      </visual>
-    </link>
-    <joint name="${prefix}housing_joint" type="fixed">
-      <parent link="${prefix}tip_calib" />
-      <child link="${prefix}housing" />
-      <origin xyz="${-0.018 - 0.01 - 0.5335} 0 0" rpy="0 0 0" />
-    </joint>
-  </xacro:macro>
+    <xacro:dv_large_needle_driver_tip prefix="${prefix}" length="${length}" />
+    <xacro:dv_large_needle_driver_rod prefix="${prefix}" length="${length}" />
+    <xacro:dv_large_needle_driver_housing_xi prefix="${prefix}" />
+  </xacro:macro> <!-- dv_large_needle_driver_470006 -->
 </robot>

Commit message: Remove old world-robot calibration

File: mops_description/urdf/mops.urdf.xacro (robot description, xacro)
@@ -1,5 +1,5 @@
 <?xml version="1.0"?>
 <robot name="mops" xmlns:xacro="http://ros.org/wiki/xacro">
-  <xacro:include filename="$(find ur_description)/urdf/ur_macro.xacro" /> <!-- From 'ros-humble-ur-description' -->
+  <xacro:include filename="$(find ur_description)/urdf/ur_macro.xacro" /> <!-- From 'ros-<distro>-ur-description' -->
   <xacro:include filename="$(find mops_description)/urdf/dv_tools.urdf.xacro" />
   <xacro:arg name="a_joint_limit_params_file" default="$(find ur_description)/config/ur5e/joint_limits.yaml" />
@@ -11,10 +11,6 @@
   <xacro:arg name="b_physical_params_file" default="$(find ur_description)/config/ur5/physical_parameters.yaml" />
   <xacro:arg name="b_visual_params_file" default="$(find ur_description)/config/ur5/visual_parameters.yaml" />
-  <!-- <xacro:arg name="world_calib_file" default="" /> -->
-  <xacro:property name="world_calib_file_prop" value="$(arg world_calib_file)" />
-  <xacro:property name="world_calib_data" value="${load_yaml(world_calib_file_prop)}" />
   <link name="world" />
   <!-- A) UR5e robot -->
-  <xacro:property name="world_to_a_base_link" value="${world_calib_data['world_to_a_base_link']}" />
   <xacro:ur_robot
       name="ur_a"
@@ -26,6 +22,5 @@
       visual_parameters_file="$(arg a_visual_params_file)"
       transmission_hw_interface="">
-    <origin xyz="${' '.join(str(val) for val in world_to_a_base_link['xyz'])}"
-        rpy="${' '.join(str(val) for val in world_to_a_base_link['rpy'])}" />
+    <origin xyz="-0.8 0.4 0.2" rpy="0 0 ${pi/2}" />
   </xacro:ur_robot>
   <!-- A) LND 470006 tool -->
@@ -34,5 +29,4 @@
   </xacro:dv_large_needle_driver_470006>
   <!-- B) UR5 robot -->
-  <xacro:property name="world_to_b_base_link" value="${world_calib_data['world_to_b_base_link']}" />
   <xacro:ur_robot
       name="ur_b"
@@ -44,6 +38,5 @@
       visual_parameters_file="$(arg b_visual_params_file)"
       transmission_hw_interface="">
-    <origin xyz="${' '.join(str(val) for val in world_to_b_base_link['xyz'])}"
-        rpy="${' '.join(str(val) for val in world_to_b_base_link['rpy'])}" />
+    <origin xyz="-0.8 -0.4 0.2" rpy="0 0 ${pi/2}" />
   </xacro:ur_robot>
   <!-- B) LND 420006 tool -->
