Commit message: description: Fix B tool attachment orientation

File: mops_description/urdf/mops.urdf.xacro (robot description, xacro)
@@ -26,5 +26,5 @@
   <!-- A) LND 470006 tool -->
   <xacro:dv_large_needle_driver_470006 prefix="a_tool_" parent="a_ur_flange">
-    <origin xyz="0.098 0 -0.053" rpy="0 ${pi/2} 0" /> <!-- FIXME -->
+    <origin xyz="0.098 0 -0.053" rpy="0 ${pi/2} 0" /> <!-- TODO: Measure/calibrate this value -->
   </xacro:dv_large_needle_driver_470006>
   <!-- B) UR5 robot -->
@@ -42,5 +42,5 @@
   <!-- B) LND 420006 tool -->
   <xacro:dv_large_needle_driver_420006 prefix="b_tool_" parent="b_ur_flange">
-    <origin xyz="0.095 0 -0.053" rpy="0 0 0" /> <!-- FIXME -->
+    <origin xyz="0.095 0 -0.053" rpy="${pi} 0 0" /> <!-- TODO: Measure/calibrate this value -->
   </xacro:dv_large_needle_driver_420006>
   <!-- Touch haptic devices -->

Commit message: Swap robot A and B positions at SDU
Also use new UR5e's hostname.

File: mops_description/urdf/mops.urdf.xacro (robot description, xacro)
@@ -22,5 +22,5 @@
       visual_parameters_file="$(arg a_visual_params_file)"
       transmission_hw_interface="">
-    <origin xyz="-0.8 0.4 0.2" rpy="0 0 ${pi/2}" />
+    <origin xyz="-0.8 -0.4 0.2" rpy="0 0 ${pi/2}" />
   </xacro:ur_robot>
   <!-- A) LND 470006 tool -->
@@ -38,5 +38,5 @@
       visual_parameters_file="$(arg b_visual_params_file)"
       transmission_hw_interface="">
-    <origin xyz="-0.8 -0.4 0.2" rpy="0 0 ${pi/2}" />
+    <origin xyz="-0.8 0.4 0.2" rpy="0 0 ${pi/2}" />
   </xacro:ur_robot>
   <!-- B) LND 420006 tool -->

Commit message: description: Fix touch_base frame placement

File: mops_description/urdf/mops.urdf.xacro (robot description, xacro)
@@ -45,15 +45,15 @@
   </xacro:dv_large_needle_driver_420006>
   <!-- Touch haptic devices -->
+  <link name="touch_right_base" />
   <link name="touch_left_base" />
-  <link name="touch_right_base" />
+  <joint name="world_touch_right_fixed" type="fixed">
+    <parent link="world" />
+    <child link="touch_right_base" />
+    <origin xyz="-1.0 -0.2 0.3" rpy="${pi/2} 0 ${-pi/2}" />
+  </joint>
   <joint name="world_touch_left_fixed" type="fixed">
-    <parent link="a_ur_base_link" />
+    <parent link="world" />
     <child link="touch_left_base" />
-    <origin xyz="-0.3 -0.4 0.1" rpy="${pi/2} 0 ${pi}" />
-  </joint>
-  <joint name="world_touch_right_fixed" type="fixed">
-    <parent link="b_ur_base_link" />
-    <child link="touch_right_base" />
-    <origin xyz="0.3 -0.4 0.1" rpy="${pi/2} 0 ${pi}" />
+    <origin xyz="-1.0 0.2 0.3" rpy="${pi/2} 0 ${-pi/2}" />
   </joint>
 </robot>

Commit message: description: Update tool descriptions

File: mops_description/urdf/mops.urdf.xacro (robot description, xacro)
@@ -26,5 +26,5 @@
   <!-- A) LND 470006 tool -->
   <xacro:dv_large_needle_driver_470006 prefix="a_tool_" parent="a_ur_flange">
-    <origin xyz="0.098 0 -0.053" rpy="0 ${pi/2} 0" /> <!-- TODO: Measure/calibrate this value -->
+    <origin xyz="0.095 0 -0.0525" rpy="0 ${pi/2} 0" /> <!-- Values taken from the tool adapter CAD model -->
   </xacro:dv_large_needle_driver_470006>
   <!-- B) UR5 robot -->
@@ -42,5 +42,5 @@
   <!-- B) LND 420006 tool -->
   <xacro:dv_large_needle_driver_420006 prefix="b_tool_" parent="b_ur_flange">
-    <origin xyz="0.095 0 -0.053" rpy="${pi} 0 0" /> <!-- TODO: Measure/calibrate this value -->
+    <origin xyz="0.127 0 0.053" rpy="${pi} 0 0" /> <!-- Values taken from the tool adapter CAD model -->
   </xacro:dv_large_needle_driver_420006>
   <!-- Touch haptic devices -->

File: mops_description/urdf/tool/dv_large_needle_driver.urdf.xacro (robot description, xacro)
@@ -3,5 +3,8 @@
 <robot name="dv_large_needle_driver" xmlns:xacro="http://ros.org/wiki/xacro">
   <!-- End-effector of the LND -->
-  <xacro:macro name="dv_large_needle_driver_tip" params="prefix length" >
+  <xacro:macro name="dv_large_needle_driver_shaft" params="prefix length" >
+    <!-- Distance from where the tool shaft (the dark grey part) meets the tool
+         tip (metallic part) to the roll joint origin -->
+    <xacro:property name="dist_shaft_to_roll_joint" value="0.009" />
     <link name="${prefix}rotation">
       <visual>
@@ -11,4 +14,12 @@
         </geometry>
         <material name="tip_metallic_gray" />
+      </visual>
+    </link>
+    <link name="${prefix}shaft">
+      <visual>
+        <geometry>
+          <cylinder radius="0.004" length="${length}" />
+        </geometry>
+        <material name="rod_dark_grey" />
       </visual>
     </link>
@@ -48,5 +59,5 @@
       <parent link="${prefix}base" />
       <child link="${prefix}rotation" />
-      <origin xyz="${length} 0 0" rpy="${-pi} ${-pi/2} 0" />
+      <origin xyz="${length + dist_shaft_to_roll_joint} 0 0" rpy="${-pi} ${-pi/2} 0" />
       <axis xyz="0 0 1" />
       <limit lower="${radians(-260)}" upper="${radians(260)}" effort="0.3" velocity="${2*pi}" />
@@ -63,4 +74,10 @@
       <child link="${prefix}jaw_hinge" />
       <origin xyz="0.0091 0 0" rpy="${pi/2} 0 0" />
+    </joint>
+    <!-- asdf -->
+    <joint name="${prefix}shaft_fixed" type="fixed">
+      <parent link="${prefix}rotation" />
+      <child link="${prefix}shaft" />
+      <origin xyz="0 0 ${-length/2 - dist_shaft_to_roll_joint}" rpy="0 0 0" />
     </joint>
     <!-- This is not a real physical joint, but rather yaw0 = (yaw1 - yaw2) / 2,
@@ -131,24 +148,12 @@
       <parent link="${prefix}base" />
       <child link="${prefix}housing" />
-      <origin xyz="-0.015 0 -0.019" rpy="0 0 0" /> <!-- FIXME -->
+      <origin xyz="-0.03 0 -0.02" rpy="0 0 0" />
     </joint>
   </xacro:macro> <!-- dv_large_needle_driver_housing_xi -->
-  <xacro:macro name="dv_large_needle_driver_rod" params="prefix length" >
-    <link name="${prefix}rod">
-      <visual>
-        <geometry>
-          <cylinder radius="0.004" length="${length}" />
-        </geometry>
-        <material name="rod_dark_grey" />
-      </visual>
-    </link>
-    <joint name="${prefix}rod_fixed" type="fixed">
-      <parent link="${prefix}rotation" />
-      <child link="${prefix}rod" />
-      <origin xyz="0 0 ${-length/2 - 0.01}" rpy="0 0 0" />
-    </joint>
-  </xacro:macro> <!-- dv_large_needle_driver_rod -->
   <xacro:macro name="dv_large_needle_driver_420006" params="prefix parent *origin">
-    <xacro:property name="length" value="0.4670" />
+    <!-- This number is the visible length of the tool shaft (the dark grey part).
+         Ie. the tool_base frame is placed where the shaft meets the housing).
+         Officially the tool's length is 0.4670m. -->
+    <xacro:property name="length" value="0.4225" />
     <link name="${prefix}base" />
     <joint name="${prefix}base_fixed" type="fixed">
@@ -157,10 +162,12 @@
       <child link="${prefix}base" />
     </joint>
-    <xacro:dv_large_needle_driver_tip prefix="${prefix}" length="${length}" />
-    <xacro:dv_large_needle_driver_rod prefix="${prefix}" length="${length}" />
+    <xacro:dv_large_needle_driver_shaft prefix="${prefix}" length="${length}" />
     <xacro:dv_large_needle_driver_housing_si prefix="${prefix}" />
   </xacro:macro> <!-- dv_large_needle_driver_420006 -->
   <xacro:macro name="dv_large_needle_driver_470006" params="prefix parent *origin">
-    <xacro:property name="length" value="0.5335" />
+    <!-- This number is the visible length of the tool shaft (the dark grey part).
+         Ie. the tool_base frame is placed where the shaft meets the housing).
+         Officially the tool's length is 0.5335m. -->
+    <xacro:property name="length" value="0.5365" />
     <link name="${prefix}base" />
     <joint name="${prefix}base_fixed" type="fixed">
@@ -169,6 +176,5 @@
       <child link="${prefix}base" />
     </joint>
-    <xacro:dv_large_needle_driver_tip prefix="${prefix}" length="${length}" />
-    <xacro:dv_large_needle_driver_rod prefix="${prefix}" length="${length}" />
+    <xacro:dv_large_needle_driver_shaft prefix="${prefix}" length="${length}" />
     <xacro:dv_large_needle_driver_housing_xi prefix="${prefix}" />
   </xacro:macro> <!-- dv_large_needle_driver_470006 -->
