Commit message: description: Fix B tool transform sign

File: mops_description/urdf/mops_sdu.urdf.xacro (robot description, xacro)
@@ -42,5 +42,5 @@
   <!-- B) LND 420006 tool -->
   <xacro:dv_large_needle_driver_420006 prefix="b_tool_" parent="b_ur_flange">
-    <origin xyz="0.127 0 0.053" rpy="${pi} 0 0" /> <!-- Values taken from the tool adapter CAD model -->
+    <origin xyz="0.127 0 -0.053" rpy="${pi} 0 0" /> <!-- Values taken from the tool adapter CAD model -->
   </xacro:dv_large_needle_driver_420006>
   <!-- Touch haptic devices -->
