Commit message: description: Fix tool housing origin

File: mops_description/urdf/tool/dv_large_needle_driver.urdf.xacro (robot description, xacro)
@@ -133,5 +133,5 @@
       <parent link="${prefix}base" />
       <child link="${prefix}housing" />
-      <origin xyz="-0.025 0 0" rpy="0 0 0" /> <!-- FIXME -->
+      <origin xyz="-0.048 0 0" rpy="0 0 0" />
     </joint>
   </xacro:macro> <!-- dv_large_needle_driver_housing_si -->
